Commit message: ok

File: catkin_ws/src/my_robot/urdf/my_robot.xacro (robot description, xacro)
@@ -1,5 +1,6 @@
 <?xml version='1.0'?>
-<robot name="my_robot" xmlns:xacro="http://www.ros.org/wiki/xacro">
-<xacro:include filename="$(find my_robot)/urdf/my_robot.gazebo" />
+<robot name="my_robot"
+  xmlns:xacro="http://www.ros.org/wiki/xacro">
+  <xacro:include filename="$(find my_robot)/urdf/my_robot.gazebo" />
   <link name="robot_footprint"></link>
   <joint name="robot_footprint_joint" type="fixed">
@@ -13,9 +14,5 @@
       <mass value="15.0"/>
       <origin xyz="0.0 0 0" rpy=" 0 0 0"/>
-      <inertia
-          ixx="0.1" ixy="0" ixz="0"
-          iyy="0.1" iyz="0"
-          izz="0.1"
-      />
+      <inertia ixx="0.1" ixy="0" ixz="0" iyy="0.1" iyz="0" izz="0.1" />
     </inertial>
     <collision name='collision'>
@@ -56,5 +53,5 @@
     </visual>
   </link>
-<!-- Left wheel -->
+  <!-- Left wheel -->
   <joint type="continuous" name="left_wheel_hinge">
     <origin xyz="0 0.15 0" rpy="0 0 0"/>
@@ -70,9 +67,5 @@
       <mass value="5.0"/>
       <origin xyz="0.0 0 0" rpy="0.0 1.5707 1.5707"/>
-      <inertia
-          ixx="0.1" ixy="0" ixz="0"
-          iyy="0.1" iyz="0"
-          izz="0.1"
-      />
+      <inertia ixx="0.1" ixy="0" ixz="0" iyy="0.1" iyz="0" izz="0.1" />
     </inertial>
     <collision name='left_wheel_collision'>
@@ -89,5 +82,5 @@
     </visual>
   </link>
-<!-- Right wheel -->
+  <!-- Right wheel -->
   <joint type="continuous" name="right_wheel_hinge">
     <origin xyz="0 -0.15 0" rpy="0 0 0"/>
@@ -103,9 +96,5 @@
       <mass value="5.0"/>
       <origin xyz="0.0 0 0" rpy="0.0 1.5707 1.5707"/>
-      <inertia
-          ixx="0.1" ixy="0" ixz="0"
-          iyy="0.1" iyz="0"
-          izz="0.1"
-      />
+      <inertia ixx="0.1" ixy="0" ixz="0" iyy="0.1" iyz="0" izz="0.1" />
     </inertial>
     <collision name='right_wheel_collision'>
@@ -122,5 +111,5 @@
     </visual>
   </link>
-<!-- For Camera -->
+  <!-- For Camera -->
   <joint type="fixed" name="camera_joint">
     <origin xyz="0.2 0 0" rpy="0 0 0"/>
@@ -134,9 +123,5 @@
       <mass value="0.1"/>
       <origin xyz="0 0 0" rpy=" 0 0 0"/>
-      <inertia
-          ixx="1e-6" ixy="0" ixz="0"
-          iyy="1e-6" iyz="0"
-          izz="1e-6"
-      />
+      <inertia ixx="1e-6" ixy="0" ixz="0" iyy="1e-6" iyz="0" izz="1e-6" />
     </inertial>
     <collision name='camera_collision'>
@@ -165,9 +150,5 @@
       <mass value="1e-5"/>
       <origin xyz="0 0 0" rpy=" 0 0 0"/>
-      <inertia
-          ixx="1e-6" ixy="0" ixz="0"
-          iyy="1e-6" iyz="0"
-          izz="1e-6"
-      />
+      <inertia ixx="1e-6" ixy="0" ixz="0" iyy="1e-6" iyz="0" izz="1e-6" />
     </inertial>
     <collision name='hokuyo_collision'>
@@ -184,3 +165,10 @@
     </visual>
   </link>
+  <joint name="camera_optical_joint" type="fixed">
+    <origin xyz="0 0 0" rpy="-1.5707 0 -1.5707"/>
+    <parent link="camera"/>
+    <child link="camera_link_optical"/>
+  </joint>
+  <link name="camera_link_optical">
+  </link>
 </robot>

Commit message: change robot color and shape

File: catkin_ws/src/my_robot/urdf/my_robot.xacro (robot description, xacro)
@@ -1,5 +1,18 @@
 <?xml version='1.0'?>
-<robot name="my_robot" xmlns:xacro="http://www.ros.org/wiki/xacro">
-<xacro:include filename="$(find my_robot)/urdf/my_robot.gazebo" />
+<robot name="my_robot"
+  xmlns:xacro="http://www.ros.org/wiki/xacro">
+  <xacro:include filename="$(find my_robot)/urdf/my_robot.gazebo" />
+  <material name="red">
+    <color rgba="0.92 0.09 0.09 1"/>
+  </material>
+  <material name="grey">
+    <color rgba="0.2 0.2 0.2 1"/>
+  </material>
+  <material name="blue">
+    <color rgba="0.13 0.65 0.70 1"/>
+  </material>
+  <material name="skyblue">
+    <color rgba="0.49 0.84 0.87 1"/>
+  </material>
   <link name="robot_footprint"></link>
   <joint name="robot_footprint_joint" type="fixed">
@@ -13,9 +26,5 @@
       <mass value="15.0"/>
       <origin xyz="0.0 0 0" rpy=" 0 0 0"/>
-      <inertia
-          ixx="0.1" ixy="0" ixz="0"
-          iyy="0.1" iyz="0"
-          izz="0.1"
-      />
+      <inertia ixx="0.1" ixy="0" ixz="0" iyy="0.1" iyz="0" izz="0.1" />
     </inertial>
     <collision name='collision'>
@@ -30,4 +39,5 @@
         <box size=".4 .2 .1"/>
       </geometry>
+      <material name="blue"/>
     </visual>
     <collision name='back_caster_collision'>
@@ -42,4 +52,5 @@
         <sphere radius="0.05"/>
       </geometry>
+      <material name="red"/>
     </visual>
     <collision name='front_caster_collision'>
@@ -54,7 +65,8 @@
         <sphere radius="0.05"/>
       </geometry>
-    </visual>
-  </link>
-<!-- Left wheel -->
+      <material name="red"/>
+    </visual>
+  </link>
+  <!-- Left wheel -->
   <joint type="continuous" name="left_wheel_hinge">
     <origin xyz="0 0.15 0" rpy="0 0 0"/>
@@ -70,9 +82,5 @@
       <mass value="5.0"/>
       <origin xyz="0.0 0 0" rpy="0.0 1.5707 1.5707"/>
-      <inertia
-          ixx="0.1" ixy="0" ixz="0"
-          iyy="0.1" iyz="0"
-          izz="0.1"
-      />
+      <inertia ixx="0.1" ixy="0" ixz="0" iyy="0.1" iyz="0" izz="0.1" />
     </inertial>
     <collision name='left_wheel_collision'>
@@ -87,7 +95,8 @@
         <cylinder radius="0.1" length="0.05"/>
       </geometry>
-    </visual>
-  </link>
-<!-- Right wheel -->
+      <material name="gray"/>
+    </visual>
+  </link>
+  <!-- Right wheel -->
   <joint type="continuous" name="right_wheel_hinge">
     <origin xyz="0 -0.15 0" rpy="0 0 0"/>
@@ -103,9 +112,5 @@
       <mass value="5.0"/>
       <origin xyz="0.0 0 0" rpy="0.0 1.5707 1.5707"/>
-      <inertia
-          ixx="0.1" ixy="0" ixz="0"
-          iyy="0.1" iyz="0"
-          izz="0.1"
-      />
+      <inertia ixx="0.1" ixy="0" ixz="0" iyy="0.1" iyz="0" izz="0.1" />
     </inertial>
     <collision name='right_wheel_collision'>
@@ -120,7 +125,8 @@
         <cylinder radius="0.1" length="0.05"/>
       </geometry>
-    </visual>
-  </link>
-<!-- For Camera -->
+      <material name="gray"/>
+    </visual>
+  </link>
+  <!-- For Camera -->
   <joint type="fixed" name="camera_joint">
     <origin xyz="0.2 0 0" rpy="0 0 0"/>
@@ -134,9 +140,5 @@
       <mass value="0.1"/>
       <origin xyz="0 0 0" rpy=" 0 0 0"/>
-      <inertia
-          ixx="1e-6" ixy="0" ixz="0"
-          iyy="1e-6" iyz="0"
-          izz="1e-6"
-      />
+      <inertia ixx="1e-6" ixy="0" ixz="0" iyy="1e-6" iyz="0" izz="1e-6" />
     </inertial>
     <collision name='camera_collision'>
@@ -165,9 +167,5 @@
       <mass value="1e-5"/>
       <origin xyz="0 0 0" rpy=" 0 0 0"/>
-      <inertia
-          ixx="1e-6" ixy="0" ixz="0"
-          iyy="1e-6" iyz="0"
-          izz="1e-6"
-      />
+      <inertia ixx="1e-6" ixy="0" ixz="0" iyy="1e-6" iyz="0" izz="1e-6" />
     </inertial>
     <collision name='hokuyo_collision'>
@@ -184,3 +182,47 @@
     </visual>
   </link>
+  <!-- For Accesory -->
+  <joint type="fixed" name="acc_01_joint">
+    <origin xyz="-0.2 0.1 0.1" rpy="0 0 0"/>
+    <child link="acc_01"/>
+    <parent link="chassis"/>
+    <axis xyz="0 1 0" rpy="0 0 0"/>
+  </joint>
+  <link name="acc_01">
+    <pose>0 0 0 0 0 0</pose>
+    <inertial>
+      <mass value="0.1"/>
+      <origin xyz="0 0 0" rpy=" 0 0 0"/>
+      <inertia ixx="1e-6" ixy="0" ixz="0" iyy="1e-6" iyz="0" izz="1e-6" />
+    </inertial>
+    <visual name='acc_01_visual'>
+      <origin xyz="0.0 0.0 0.0" rpy="0.0 0 0"/>
+      <geometry>
+        <cylinder radius="0.01" length="0.2"/>
+      </geometry>
+      <material name="skyblue"/>
+    </visual>
+  </link>
+  <!-- For Accesory -->
+  <joint type="fixed" name="acc_02_joint">
+    <origin xyz="-0.2 -0.1 0.1" rpy="0 0 0"/>
+    <child link="acc_02"/>
+    <parent link="chassis"/>
+    <axis xyz="0 1 0" rpy="0 0 0"/>
+  </joint>
+  <link name="acc_02">
+    <pose>0 0 0 0 0 0</pose>
+    <inertial>
+      <mass value="0.1"/>
+      <origin xyz="0 0 0" rpy=" 0 0 0"/>
+      <inertia ixx="1e-6" ixy="0" ixz="0" iyy="1e-6" iyz="0" izz="1e-6" />
+    </inertial>
+    <visual name='acc_02_visual'>
+      <origin xyz="0.0 0.0 0.0" rpy="0.0 0 0"/>
+      <geometry>
+        <cylinder radius="0.01" length="0.2"/>
+      </geometry>
+      <material name="skyblue"/>
+    </visual>
+  </link>
 </robot>

Commit message: create WS

File: catkin_ws/src/my_robot/urdf/my_robot.xacro (robot description, xacro)
@@ -3,4 +3,16 @@
   xmlns:xacro="http://www.ros.org/wiki/xacro">
   <xacro:include filename="$(find my_robot)/urdf/my_robot.gazebo" />
+  <material name="red">
+    <color rgba="0.92 0.09 0.09 1"/>
+  </material>
+  <material name="grey">
+    <color rgba="0.2 0.2 0.2 1"/>
+  </material>
+  <material name="blue">
+    <color rgba="0.13 0.65 0.70 1"/>
+  </material>
+  <material name="skyblue">
+    <color rgba="0.49 0.84 0.87 1"/>
+  </material>
   <link name="robot_footprint"></link>
   <joint name="robot_footprint_joint" type="fixed">
@@ -27,4 +39,5 @@
         <box size=".4 .2 .1"/>
       </geometry>
+      <material name="blue"/>
     </visual>
     <collision name='back_caster_collision'>
@@ -39,4 +52,5 @@
         <sphere radius="0.05"/>
       </geometry>
+      <material name="red"/>
     </visual>
     <collision name='front_caster_collision'>
@@ -51,4 +65,5 @@
         <sphere radius="0.05"/>
       </geometry>
+      <material name="red"/>
     </visual>
   </link>
@@ -80,4 +95,5 @@
         <cylinder radius="0.1" length="0.05"/>
       </geometry>
+      <material name="gray"/>
     </visual>
   </link>
@@ -109,4 +125,5 @@
         <cylinder radius="0.1" length="0.05"/>
       </geometry>
+      <material name="gray"/>
     </visual>
   </link>
@@ -165,10 +182,47 @@
     </visual>
   </link>
-  <joint name="camera_optical_joint" type="fixed">
-    <origin xyz="0 0 0" rpy="-1.5707 0 -1.5707"/>
-    <parent link="camera"/>
-    <child link="camera_link_optical"/>
-  </joint>
-  <link name="camera_link_optical">
+  <!-- For Accesory -->
+  <joint type="fixed" name="acc_01_joint">
+    <origin xyz="-0.2 0.1 0.1" rpy="0 0 0"/>
+    <child link="acc_01"/>
+    <parent link="chassis"/>
+    <axis xyz="0 1 0" rpy="0 0 0"/>
+  </joint>
+  <link name="acc_01">
+    <pose>0 0 0 0 0 0</pose>
+    <inertial>
+      <mass value="0.1"/>
+      <origin xyz="0 0 0" rpy=" 0 0 0"/>
+      <inertia ixx="1e-6" ixy="0" ixz="0" iyy="1e-6" iyz="0" izz="1e-6" />
+    </inertial>
+    <visual name='acc_01_visual'>
+      <origin xyz="0.0 0.0 0.0" rpy="0.0 0 0"/>
+      <geometry>
+        <cylinder radius="0.01" length="0.2"/>
+      </geometry>
+      <material name="skyblue"/>
+    </visual>
+  </link>
+  <!-- For Accesory -->
+  <joint type="fixed" name="acc_02_joint">
+    <origin xyz="-0.2 -0.1 0.1" rpy="0 0 0"/>
+    <child link="acc_02"/>
+    <parent link="chassis"/>
+    <axis xyz="0 1 0" rpy="0 0 0"/>
+  </joint>
+  <link name="acc_02">
+    <pose>0 0 0 0 0 0</pose>
+    <inertial>
+      <mass value="0.1"/>
+      <origin xyz="0 0 0" rpy=" 0 0 0"/>
+      <inertia ixx="1e-6" ixy="0" ixz="0" iyy="1e-6" iyz="0" izz="1e-6" />
+    </inertial>
+    <visual name='acc_02_visual'>
+      <origin xyz="0.0 0.0 0.0" rpy="0.0 0 0"/>
+      <geometry>
+        <cylinder radius="0.01" length="0.2"/>
+      </geometry>
+      <material name="skyblue"/>
+    </visual>
   </link>
 </robot>
